Commit message: update world

File: ackermann_vehicle_description/urdf/ackermann.urdf.xacro (robot description, xacro)
@@ -1,7 +1,4 @@
 <?xml version="1.0"?>
-<!--
-Modified from em_3905 model from Wunderkammer Lab
--->
-<robot name="em_3905" xmlns:xacro="http://www.ros.org/wiki/xacro">
+<robot name="ackermann" xmlns:xacro="http://www.ros.org/wiki/xacro">
   <!-- Degree-to-radian conversions -->
   <xacro:property name="degrees_45" value="0.785398163"/>
@@ -38,16 +35,4 @@
   <xacro:property name="shock_eff_limit" value="12.5106"/>
   <xacro:property name="shock_vel_limit" value="1000"/>
-  <!-- The specifications for a Titan(R) 550 motor could not be found, so the
-       stall torque of a Mabuchi Motor(R) RS-550VC-7525 motor was used instead.
-       num_spur_gear_teeth = 68
-       num_pinion_gear_teeth = 19
-       final_gear_ratio = (num_spur_gear_teeth / num_pinion_gear_teeth) *
-         5.22 = 18.68
-       stall_torque = 0.549 N m
-       axle_eff_limit = ((2 * stall_torque) * final_gear_ratio) / 4 =
-         5.12766 N m
-       max_speed = 40 mph (30+ mph) = 17.8816 m/s
-       axle_vel_limit = (2 * pi) * (max_speed / (pi * tire_dia)) =
-         244.8696 rad/s -->
   <xacro:property name="axle_eff_limit" value="5.12766"/>
   <xacro:property name="axle_vel_limit" value="244.8696"/>
@@ -58,5 +43,5 @@
   <xacro:property name="servo_no_load_speed" value="4.553"/>
   <material name="chassis_mat">
-    <color rgba="0 0 0 1"/>
+    <color rgba="0 0 1 1"/>
   </material>
   <material name="tire_mat">
@@ -257,5 +242,5 @@
   </link>
   <gazebo reference="chassis">
-    <material>Gazebo/White</material>
+    <material>Gazebo/Blue</material>
   </gazebo>
   <joint name="base_link_to_chassis" type="fixed">
